File: PCB/MacroPad.kicad_pcb (KiCad board)
At the start: 2 copper layers, 98.8 x 95.7 mm, 34 parts, among them J1 OLED_DISPLAY, SW1 SW_Push, SW10 SW_Push, SW11 SW_Push, SW13 RotaryEncoder_Switch, SW14 RotaryEncoder_Switch, SW15 SW_Push, SW2 SW_Push, SW3 SW_Push, SW4 SW_Push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

Commit message: a
Parts:
- removed D15: 1N4148WT, Diode_SMD:D_SOD-523
- added D12: 1N914, Diode_THT:D_DO-35_SOD27_P7.62mm_Horizontal, F.Cu at (125.9, 137.2)
- D1, D10, D11, D13, D14, D2, D3, D4, D5, D6, D7, D8, D9: value 1N4148WT -> 1N914; footprint Diode_SMD:D_SOD-523 -> Diode_THT:D_DO-35_SOD27_P7.62mm_Horizontal; moved to F.Cu
- J1: value OLED_DISPLAY -> (none)
- moved D14 57.4 mm to (172.2, 86.6)
- moved D6 50.0 mm to (125.8, 103.9)
- moved D13 37.5 mm to (146.7, 122.6), turned to -90 degrees
- moved D3 36.5 mm to (125.8, 84.9)
- moved D11 28.3 mm to (106.8, 142.0)
- moved D5 28.1 mm to (106.8, 103.9)
- moved D10 27.4 mm to (87.8, 142.1)
- moved D1 26.8 mm to (87.8, 84.9)
- moved D4 26.5 mm to (87.7, 103.9)
- moved D2 26.2 mm to (106.8, 85.0)
- moved D7 8.67 mm to (87.8, 123.1)
- moved D8 8.47 mm to (106.8, 123.1)
- moved D9 7.49 mm to (125.9, 123.0)
Connections:
- D13 pad 1: Row 1 -> Row 4
- D13 pad 2: EC11SWA -> EC11SWC
- D14 pad 1: Row 4 -> Row 1
- D14 pad 2: EC11SWC -> EC11SWA
- D3 pad 1: EC11A -> Row 1
- D4 pad 1: EC11A -> Row 2
- D5 pad 1: EC11A -> Row 2
- D6 pad 1: Row 4 -> Row 2
- D7 pad 1: EC12A -> Row 3
- D8 pad 1: EC12A -> Row 3
- D9 pad 1: EC12A -> Row 3
- SW1 pad 2: Net-(D1-A) -> Net-(D2-A)
- SW10 pad 2: Net-(D10-A) -> Net-(D11-A)
- SW11 pad 2: Net-(D11-A) -> Net-(D12-A)
- SW13 pad A: EC11A -> unconnected-(SW13-PadA)
- SW13 pad B: Column 4 -> unconnected-(SW13-PadB)
- SW13 pad C: GND -> unconnected-(SW13-PadC)
- SW14 pad A: EC12A -> unconnected-(SW14-PadA)
- SW14 pad B: Column 4 -> unconnected-(SW14-PadB)
- SW14 pad C: GND -> unconnected-(SW14-PadC)
- SW15 pad 2: Net-(D15-A) -> Net-(D1-A)
- SW2 pad 2: Net-(D2-A) -> Net-(D3-A)
- SW3 pad 2: Net-(D3-A) -> Net-(D4-A)
- SW4 pad 2: Net-(D4-A) -> Net-(D5-A)
- SW5 pad 2: Net-(D5-A) -> Net-(D6-A)
- SW6 pad 2: Net-(D6-A) -> Net-(D10-A)
- U2 pad 10: EC11A -> Row 2
- U2 pad 9: EC12A -> Row 3
Routing:
- net EC11A: track 120.2 -> 0.00 mm
- net EC12A: track 114.8 -> 0.00 mm
- net Row 2: track 0.00 -> 93.3 mm
- net GND: track 122.3 -> 29.3 mm
- net Row 3: track 0.00 -> 91.0 mm
- net Column 4: track 121.2 -> 70.5 mm
- net Row 1: track 124.5 -> 96.7 mm
- net Row 4: track 129.5 -> 111.5 mm
- net EC11SWC: track 7.52 -> 20.9 mm
- net Column 1: track 167.9 -> 180.9 mm
- net Net-(D15-A): track 12.1 -> 0.00 mm
- net Net-(D12-A): track 0.00 -> 6.39 mm
- net Net-(D11-A): track 12.9 -> 6.98 mm
- net Net-(D5-A): track 12.8 -> 7.04 mm
- net Net-(D7-A): track 12.7 -> 7.05 mm
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- added copper zone on B.Cu, net (none)
- added copper zone on F.Cu, net (none)
Other:
- board text removed: "Seeed Studio"
- board text removed: "XIAO"

Commit message: Final
Parts:
- J1: value (none) -> OLED_DISPLAY
Connections:
- U2 pad 12: unconnected-(U2-3V3-Pad12) -> VCC
- U2 pad 14: VCC -> unconnected-(U2-5V-Pad14)
Routing:
- net VCC: track 38.2 -> 24.2 mm
Changed lines of the file:
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@@
 		(tenting front back)
 		(pcbplotparams
-			(layerselection 0x00000000_00000000_55555555_5755f5ff)
+			(layerselection 0x00000000_00000000_55557fdf_57ffffff)
 			(plot_on_all_layers_selection 0x00000000_00000000_00000000_00000000)
 			(disableapertmacros no)
 			(usegerberextensions yes)
-			(usegerberattributes no)
-			(usegerberadvancedattributes no)
+			(usegerberattributes yes)
+			(usegerberadvancedattributes yes)
 			(creategerberjobfile no)
 			(dashed_line_dash_ratio 12.000000)
@@
 			(sketchdnponfab yes)
 			(crossoutdnponfab yes)
-			(subtractmaskfromsilk yes)
+			(subtractmaskfromsilk no)
 			(outputformat 1)
 			(mirror no)
 			(drillshape 0)
 			(scaleselection 1)
-			(outputdirectory "../Production/Gerbers/")
+			(outputdirectory "../Gerbers/")
 		)
 	)
@@
 	(net 19 "Column 3")
 	(net 20 "Column 1")
-	(net 21 "unconnected-(U2-3V3-Pad12)")
+	(net 21 "unconnected-(U2-5V-Pad14)")
 	(net 22 "unconnected-(U2-GPIO0_D6_TX-Pad7)")
 	(net 23 "Row 4")
@@
 			)
 		)
-		(property "Value" ""
+		(property "Value" "OLED_DISPLAY"
 			(at 18.5 14 90)
 			(layer "F.Fab")
@@
 			(layers "*.Cu" "*.Mask")
 			(remove_unused_layers no)
-			(net 21 "unconnected-(U2-3V3-Pad12)")
+			(net 16 "VCC")
 			(pinfunction "3V3")
 			(pintype "passive")
@@
 			(layers "*.Cu" "*.Mask")
 			(remove_unused_layers no)
-			(net 16 "VCC")
+			(net 21 "unconnected-(U2-5V-Pad14)")
 			(pinfunction "5V")
 			(pintype "passive")
@@
 	)
 	(segment
-		(start 156.725 87.455)
-		(end 158.28 85.9)
-		(width 0.2)
-		(layer "F.Cu")
-		(net 16)
-	)
-	(segment
-		(start 163.1 85.9)
-		(end 163.1 98.75)
+		(start 174.677985 94.872016)
+		(end 174.677985 97.1355)
 		(width 0.2)
 		(layer "F.Cu")
@@
 	)
 	(segment
-		(start 158.28 85.9)
-		(end 163.1 85.9)
+		(start 157.876 86.304)
+		(end 166.109969 86.304)
 		(width 0.2)
 		(layer "F.Cu")
@@
 	)
 	(segment
-		(start 179.757985 98.607985)
-		(end 179.757985 97.1355)
-		(width 0.2)
-		(layer "F.Cu")
-		(net 16)
-	)
-	(segment
-		(start 179.8 98.75)
-		(end 179.85 98.7)
-		(width 0.2)
-		(layer "F.Cu")
-		(net 16)
-	)
-	(segment
-		(start 163.1 98.75)
-		(end 179.8 98.75)
+		(start 156.725 87.455)
+		(end 157.876 86.304)
 		(width 0.2)
 		(layer "F.Cu")
@@
 	)
 	(segment
-		(start 179.85 98.7)
-		(end 179.757985 98.607985)
+		(start 166.109969 86.304)
+		(end 174.677985 94.872016)
 		(width 0.2)
 		(layer "F.Cu")
@@
 		(polygon
 			(pts
-				(xy 73.5 53.5) (xy 72.45 159.6) (xy 189.45 158) (xy 191.7 48.05)
+				(xy 78.45 49.8) (xy 78.15 164.7) (xy 193.25 158.65) (xy 191.35 50.45)
 			)
 		)
