File: PCB/MacroPad.kicad_sch (KiCad schematic)
At the start: 30 parts, among them J1 OLED_DISPLAY, SW1 SW_Push, SW10 SW_Push, SW11 SW_Push, SW13 RotaryEncoder_Switch, SW14 RotaryEncoder_Switch, SW15 SW_Push, SW2 SW_Push, SW3 SW_Push, SW4 SW_Push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

Commit message: a
Parts:
- removed D1, D10, D11, D13, D14, D15, D2, D3, D4, D5, D6, D7, D8, D9: 1N4148WT, Diode_SMD:D_SOD-523, symbol Diode:1N4148WT
- added D1, D10, D11, D12, D13, D14, D2, D3, D4, D5, D6, D7, D8, D9: 1N914, Diode_THT:D_DO-35_SOD27_P7.62mm_Horizontal, symbol Diode:1N914
Connections:
- net Column 4: no longer SW13.B, SW14.B
- net EC11SWA: now also D14.2 (A)
- net EC11SWC: now also D13.2 (A)
- net GND: no longer SW13.C, SW14.C
- net Row 1: now also D1.1 (K), D14.1 (K), D2.1 (K), D3.1 (K)
- net Row 4: now also D10.1 (K), D11.1 (K), D12.1 (K), D13.1 (K)
- net at SW2.2: now also D3.2 (A)
- net at SW3.2: now also D4.2 (A)
- net at SW10.2: now also D11.2 (A)
- net at SW15.2: now also D1.2 (A)
- net at SW8.2: now also D8.2 (A)
- net at SW5.2: now also D6.2 (A)
- net at SW6.2: now also D10.2 (A)
- net at SW11.2: now also D12.2 (A)
- net at SW9.2: now also D9.2 (A)
- net at SW1.2: now also D2.2 (A)
- net at SW7.2: now also D7.2 (A)
- net at SW4.2: now also D5.2 (A)
- net EC11A: no longer names the net of SW13.A
- net EC11A: no longer U2.10 (GPIO4_D9_MISO)
- net EC12A: no longer names the net of SW14.A
- net EC12A: no longer U2.9 (GPIO2_D8_SCK)
- new net Row 2: D4.1 (K), D5.1 (K), D6.1 (K), U2.10 (GPIO4_D9_MISO)
- new net Row 3: D7.1 (K), D8.1 (K), D9.1 (K), U2.9 (GPIO2_D8_SCK)

Commit message: Final
Connections:
- net VCC: now also U2.12 (3V3); no longer U2.14 (5V)
Changed lines of the file:
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@@
-	(wire
-		(pts
-			(xy 222.25 33.02) (xy 229.87 33.02)
-		)
-		(stroke
-			(width 0)
-			(type default)
-		)
-	)
 	(wire
 		(pts
@@
 	(wire
 		(pts
-			(xy 222.25 29.21) (xy 228.6 29.21)
-		)
-		(stroke
-			(width 0)
-			(type default)
-		)
-	)
-	(wire
-		(pts
 			(xy 77.47 77.47) (xy 93.98 77.47)
 		)
@@
 	(wire
 		(pts
+			(xy 222.25 33.02) (xy 224.79 33.02)
+		)
+		(stroke
+			(width 0)
+			(type default)
+		)
+	)
+	(wire
+		(pts
 			(xy 39.37 33.02) (xy 39.37 41.91)
 		)
@@
 		(pts
 			(xy 124.46 45.72) (xy 120.65 45.72)
+		)
+		(stroke
+			(width 0)
+			(type default)
+		)
+	)
+	(wire
+		(pts
+			(xy 222.25 36.83) (xy 229.87 36.83)
 		)
 		(stroke
@@
 	(symbol
 		(lib_id "power:VCC")
-		(at 228.6 29.21 0)
+		(at 229.87 36.83 0)
 		(unit 1)
 		(exclude_from_sim no)
@@
 		(fields_autoplaced yes)
 		(property "Reference" "#PWR02"
-			(at 228.6 33.02 0)
+			(at 229.87 40.64 0)
 			(effects
 				(font
@@
 		)
 		(property "Value" "VCC"
-			(at 228.6 24.13 0)
+			(at 229.87 31.75 0)
 			(effects
 				(font
@@
 		)
 		(property "Footprint" ""
-			(at 228.6 29.21 0)
+			(at 229.87 36.83 0)
 			(effects
 				(font
@@
 		)
 		(property "Datasheet" ""
-			(at 228.6 29.21 0)
+			(at 229.87 36.83 0)
 			(effects
 				(font
@@
 		)
 		(property "Description" "Power symbol creates a global label with name \"VCC\""
-			(at 228.6 29.21 0)
+			(at 229.87 36.83 0)
 			(effects
 				(font
@@
 	(symbol
 		(lib_id "power:GND")
-		(at 229.87 33.02 0)
+		(at 224.79 33.02 180)
 		(unit 1)
 		(exclude_from_sim no)
@@
 		(fields_autoplaced yes)
 		(property "Reference" "#PWR07"
-			(at 229.87 39.37 0)
+			(at 224.79 26.67 0)
 			(effects
 				(font
@@
 		)
 		(property "Value" "GND"
-			(at 229.87 38.1 0)
+			(at 224.79 27.94 0)
 			(effects
 				(font
@@
 		)
 		(property "Footprint" ""
-			(at 229.87 33.02 0)
+			(at 224.79 33.02 0)
 			(effects
 				(font
@@
 		)
 		(property "Datasheet" ""
-			(at 229.87 33.02 0)
+			(at 224.79 33.02 0)
 			(effects
 				(font
@@
 		)
 		(property "Description" "Power symbol creates a global label with name \"GND\" , ground"
-			(at 229.87 33.02 0)
-			(effects
-				(font
+			(at 224.79 33.02 0)
+			(effects
+				(font
